File: kicad7.0/Octopus2CPAP.kicad_sch (KiCad schematic)
At the start: 9 parts, among them J1 Conn_02x05_Odd_Even, J2 Conn_01x02_Pin, Q1 AO3400A, U1 74LVC1G125

Commit message: finalize and release
Parts:
- removed JP1: Jumper_2_Bridged, Jumper:SolderJumper-2_P1.3mm_Bridged_RoundedPad1.0x1.5mm, symbol Jumper:Jumper_2_Bridged
- added R4: 10R, Resistor_SMD:R_0805_2012Metric_Pad1.20x1.40mm_HandSolder, symbol Device:R
- BZ1, J1, J2: now left out of the parts list
- Q1: JLCPCB Rotation Offset (none) -> 180; MPN (none) -> C20917
- R1: MPN (none) -> C17673
- R2: value 330 -> 300R; MPN (none) -> C17617
- R3: MPN (none) -> C17414
- U1: footprint Package_TO_SOT_SMD:SOT-353_SC-70-5_Handsoldering -> Package_TO_SOT_SMD:SOT-23-5_HandSoldering; JLCPCB Rotation Offset (none) -> -90; MPN (none) -> C23654
Connections:
- net +5V: now also R4.2; no longer BZ1.1 (-)
- net BEEPER_H: now also BZ1.2 (+)
- new net: BZ1.1 (-), R4.1
Other:
- moved on the sheet: J1
